File: LattePanda_Module.kicad_sch (KiCad schematic)
At the start: 0 parts

Commit message: Started with the LattePanda module. Unconnected and some other various initial configs
Parts:
- added A78: LattePanda_Mu, Module_LattePanda:LattePanda_Module_H8.0mm_Horizontal, symbol MCU_Module_LattePanda:LattePanda_Mu
- added R2: 10k/1%, symbol Device:R
- added TP78: TestPoint, symbol Connector:TestPoint
Connections:
- new net: A78.133 (~{BIOS_SEL}), R2.1, TP78.1
- new net: A78.250 (VIN), A78.251 (VIN), A78.252 (VIN), A78.253 (VIN), A78.254 (VIN), A78.255 (VIN), A78.256 (VIN), A78.257 (VIN), A78.258 (VIN), A78.259 (VIN), A78.260 (VIN)
- new net GND: A78.101 (GND), A78.107 (GND), A78.11 (GND), A78.110 (GND), A78.113 (GND), A78.116 (GND), A78.135 (GND), A78.136 (GND), A78.14 (GND), A78.151 (GND), A78.158 (GND), A78.167 (GND), A78.17 (GND), A78.170 (GND), A78.181 (GND), A78.182 (GND), A78.188 (GND), A78.189 (GND), A78.194 (GND), A78.195 (GND), A78.20 (GND), A78.200 (GND), A78.201 (GND), A78.206 (GND), A78.207 (GND), A78.212 (GND), A78.213 (GND), A78.218 (GND), A78.219 (GND), A78.224 (GND), A78.225 (GND), A78.23 (GND), A78.230 (GND), A78.231 (GND), A78.236 (GND), A78.237 (GND), A78.242 (GND), A78.243 (GND), A78.248 (GND), A78.249 (GND), A78.26 (GND), A78.29 (GND), A78.32 (GND), A78.35 (GND), A78.38 (GND), A78.41 (GND), A78.44 (GND), A78.47 (GND), A78.50 (GND), A78.53 (GND), A78.56 (GND), A78.59 (GND), A78.62 (GND), A78.65 (GND), A78.68 (GND), A78.71 (GND), A78.74 (GND), A78.77 (GND), A78.80 (GND), A78.83 (GND), A78.86 (GND), A78.89 (GND), A78.92 (GND), A78.95 (GND), A78.98 (GND), A78.MP (Mountinge_Pads)
- new net VPullup: R2.2
- no-connect marks 0 -> 84
