File: LattePanda_Module.kicad_sch (KiCad schematic)
At the start: 12 parts, among them J78 Conn_01x03_Pin

Commit message: Started on physical placement of components but footprint got H6 is incoorect. Schematic needs annotation before importing the changes.
Parts:
- H6: footprint A_HDJ_Library:MountingHole_3.2mm_M3_Pad_Via -> A_HDJ_Library:MountingHole_3mm_M2_Pad_TopOnly
Changed lines of the file:
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@@
 			)
 		)
-		(property "Footprint" "A_HDJ_Library:MountingHole_3.2mm_M3_Pad_Via"
+		(property "Footprint" "A_HDJ_Library:MountingHole_3mm_M2_Pad_TopOnly"
 			(at 470.408 302.26 0)
 			(hide yes)
