File: PSU.kicad_sch (KiCad schematic)
At the start: 84 parts, among them J17 Barrel_Jack_Switch, J18 USB_C_Receptacle_USB2.0_16P, Q5 2N7002, Q78 AON7262E, Q79 2N7002, Q80 2N7002, SW1 SW_Push, SW2 SW_Push, U13 TL431DBZ, U14 USB PD等快充协议受电芯片-CH224K-ESSOP10, U15 LM2734X, U16 LM2734X

Commit message: Fixed the Grid connection errors in the PSU Schematic sheet
Parts:
- added TP9: TestPoint, symbol Connector:TestPoint
- renumbered R51 to R46, R52 to R53, R46 to R54
Connections:
- net +12VA: now also C63.2, Q78.4 (G), R44.2, R45.2
- net +15V: now also D18.2 (A), D19.2 (A), D20.2 (A), R37.1, TP3.1
- net VDC: no longer C63.1, Q78.1 (S_1), Q78.2 (S_2), Q78.3 (S_3), R38.2, R40.2, R44.1
- net at Q80.1 (G): now also TP9.1
- net at R59.1, R60.2: now also U16.3 (FB)
- new net: C63.1, Q78.1 (S_1), Q78.2 (S_2), Q78.3 (S_3), R38.2, R40.2, R44.1
Other:
- moved on the sheet: C61, C62, C63, C64, C65, C66, C67, C68, C69, C70, C71, C74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

Commit message: Added the ESSOP official footprint for the IC in the PSU sheet that was missing
Parts:
- U14: footprint ESSOP10 -> A_HDJ_Library:ESSOP-10-1EP_3.9x5mm_P1.0mm_EP3.2x2.3
Changed lines of the file:
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@@
 			)
 		)
-		(property "Footprint" "ESSOP10"
+		(property "Footprint" "A_HDJ_Library:ESSOP-10-1EP_3.9x5mm_P1.0mm_EP3.2x2.3"
 			(at 189.23 262.89 0)
 			(hide yes)

Commit message: Updated all the footprints into the pcb editor but all the designator numbers have changed... I have tp go back and fix each one
Parts:
- J18: footprint (none) -> A_HDJ_Library:USB_C_Receptacle_G-Switch_GT-USB-7010ASV
- JP78: footprint (none) -> A_HDJ_Library:PinHeader_1x03_P2.54mm_Vertical
- R100: renamed from R54; footprint (none) -> A_HDJ_Library:R_0402_1005Metric
- R86: renamed from R38; footprint (none) -> A_HDJ_Library:R_0402_1005Metric
- R87: renamed from R39; footprint (none) -> A_HDJ_Library:R_0402_1005Metric
- R88: renamed from R40; footprint (none) -> A_HDJ_Library:R_0402_1005Metric
- R89: renamed from R43; footprint (none) -> A_HDJ_Library:R_0402_1005Metric
- R90: renamed from R41; footprint (none) -> A_HDJ_Library:R_0402_1005Metric
- R91: renamed from R44; footprint (none) -> A_HDJ_Library:R_0402_1005Metric
- R92: renamed from R42; footprint (none) -> A_HDJ_Library:R_0402_1005Metric
- R93: renamed from R45; footprint (none) -> A_HDJ_Library:R_0402_1005Metric
- TP79: renamed from TP4; footprint (none) -> A_HDJ_Library:TestPoint_Pad_D1.5mm
- TP80: renamed from TP3; footprint (none) -> A_HDJ_Library:TestPoint_Pad_D1.5mm
- TP81: renamed from TP10; footprint (none) -> A_HDJ_Library:TestPoint_Pad_D1.5mm
- TP82: renamed from TP9; footprint (none) -> A_HDJ_Library:TestPoint_Pad_D1.5mm
- TP83: renamed from TP8; footprint (none) -> A_HDJ_Library:TestPoint_Pad_D1.5mm
- TP84: renamed from TP13; footprint (none) -> A_HDJ_Library:TestPoint_Pad_D1.5mm
- TP85: renamed from TP5; footprint (none) -> A_HDJ_Library:TestPoint_Pad_D1.5mm
- TP86: renamed from TP6; footprint (none) -> A_HDJ_Library:TestPoint_Pad_D1.5mm
- U14: value USB PD等快充协议受电芯片-CH224K-ESSOP10 -> CH224K
- renumbered C61 to C78, C63 to C79, C62 to C80, C66 to C81, C64 to C82, C65 to C83, C68 to C84, C67 to C85, C69 to C86, C70 to C87, C71 to C88, C74 to C89, C75 to C90, C76 to C91, C77 to C92, C78 to C93, C79 to C94, C80 to C95, C81 to C96, C82 to C97, C83 to C98, D10 to D78, D11 to D79, D12 to D80, D13 to D81, D14 to D82, D15 to D83, D16 to D84, D17 to D85, D18 to D86, D19 to D87, D20 to D88, D21 to D89, D78 to D90, D22 to D91, D79 to D92, D25 to D93, J17 to J80, L1 to L78, L2 to L79, Q5 to Q78, Q80 to Q79, Q78 to Q80, Q79 to Q81, R52 to R101, R51 to R102, R55 to R103, R56 to R104, R59 to R105, R60 to R106, R57 to R107, R58 to R108, R36 to R84, R37 to R85, R48 to R94, R50 to R95, R47 to R96, R49 to R97, R46 to R98, R53 to R99, SW1 to SW78, SW2 to SW79, U13 to U79, U15 to U80, U16 to U81

Commit message: Designators in PSU restored
Parts:
- renumbered C78 to C61, C79 to C63, C82 to C64, C83 to C65, C85 to C66, C81 to C66, C84 to C67, C86 to C69, C87 to C70, C88 to C71, C89 to C74, C90 to C75, C91 to C76, C92 to C77, C93 to C78, C94 to C79, C95 to C80, C96 to C81, C97 to C82, C98 to C83, D78 to D10, D79 to D11, D80 to D12, D81 to D13, D82 to D14, D83 to D15, D84 to D16, D85 to D17, D86 to D18, D87 to D19, D88 to D20, D89 to D21, D91 to D22, D92 to D24, D93 to D25, J80 to J17, JP78 to JP1, L78 to L1, L79 to L2, Q80 to Q7, Q81 to Q8, R84 to R36, R85 to R37, R89 to R43, R91 to R44, R98 to R46, R96 to R47, R97 to R49, R95 to R50, R102 to R51, R101 to R52, R99 to R53, R103 to R55, R104 to R56, R107 to R57, R108 to R58, R105 to R59, R106 to R60, R94 to R66, SW78 to SW1, SW79 to SW2, TP84 to TP13, TP80 to TP3, TP79 to TP4, TP85 to TP5, TP86 to TP6, TP83 to TP8, TP82 to TP9, U80 to U15, U81 to U16
Connections:
- net +12V: now also C63.1, Q7.1 (S_1), Q7.2 (S_2), Q7.3 (S_3), R44.1, R86.2, R88.2
- net +12VA: no longer C63.2, Q7.4 (G), R44.2, R93.2
- new net: C63.2, Q7.4 (G), R44.2, R93.2
