File: Fan.kicad_sch (KiCad schematic)
At the start: 23 parts, among them M1 Fan_4pin, M2 Fan_4pin

Commit message: Resolved some duplicate annotations
Parts:
- renumbered R66 to R206
Changed lines of the file:
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@@
 		(in_pos_files yes)
 		(dnp no)
-		(property "Reference" "R66"
+		(property "Reference" "R206"
 			(at 169.672 69.85 90)
 			(show_name no)
@@
 			(project "Carrier_Board"
 				(path "/e768274e-12f3-4f83-96f6-abb7638e0bc1/db5534e0-ad9a-443b-b9b9-b696f6fb2c85"
-					(reference "R66")
+					(reference "R206")
 					(unit 1)
 				)
