File: hdmi.kicad_sch (KiCad schematic)
At the start: 37 parts, among them J3 HDMI_A, Q1 2N7002, Q2 2SK3018, Q3 2SK3018, Q85 2SK3018, U1 D3V3XA4B10LP, U2 D3V3XA4B10LP

Commit message: Resolved some duplicate annotations
Parts:
- renumbered C27 to C24
Changed lines of the file:
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@@
 		(in_pos_files yes)
 		(dnp no)
-		(property "Reference" "C27"
+		(property "Reference" "C24"
 			(at 141.478 57.15 90)
 			(show_name no)
@@
 			(project "Carrier_Board"
 				(path "/e768274e-12f3-4f83-96f6-abb7638e0bc1/1c6e1139-d819-4324-bacb-4e7c941be195"
-					(reference "C27")
+					(reference "C24")
 					(unit 1)
 				)

Commit message: Created new Heiarchal sheet for audio, and started to arrange passive components for the HDMI connector
Parts:
- renumbered Q85 to Q4, R143 to R19
Changed lines of the file:
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@@
 		(in_pos_files yes)
 		(dnp no)
-		(property "Reference" "R143"
+		(property "Reference" "R19"
 			(at 198.374 101.6 90)
 			(show_name no)
@@
 			(project "Carrier_Board"
 				(path "/e768274e-12f3-4f83-96f6-abb7638e0bc1/1c6e1139-d819-4324-bacb-4e7c941be195"
-					(reference "R143")
+					(reference "R19")
 					(unit 1)
 				)
@@
 		(in_pos_files yes)
 		(dnp no)
-		(property "Reference" "Q85"
+		(property "Reference" "Q4"
 			(at 182.88 101.5999 0)
 			(show_name no)
@@
 			(project "Carrier_Board"
 				(path "/e768274e-12f3-4f83-96f6-abb7638e0bc1/1c6e1139-d819-4324-bacb-4e7c941be195"
-					(reference "Q85")
+					(reference "Q4")
 					(unit 1)
 				)

Commit message: Optimized tracks around Ethernet and repaird the HDMI circuit from component skew memory leak
Parts:
- renumbered R132 to R15, R134 to R18
Changed lines of the file:
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@@
 		(in_pos_files yes)
 		(dnp no)
-		(property "Reference" "R132"
+		(property "Reference" "R15"
 			(at 127.762 97.028 0)
 			(show_name no)
@@
 			(project "Carrier_Board"
 				(path "/e768274e-12f3-4f83-96f6-abb7638e0bc1/1c6e1139-d819-4324-bacb-4e7c941be195"
-					(reference "R132")
+					(reference "R15")
 					(unit 1)
 				)
@@
 		(in_pos_files yes)
 		(dnp no)
-		(property "Reference" "R134"
+		(property "Reference" "R18"
 			(at 137.922 97.028 0)
 			(show_name no)
@@
 			(project "Carrier_Board"
 				(path "/e768274e-12f3-4f83-96f6-abb7638e0bc1/1c6e1139-d819-4324-bacb-4e7c941be195"
-					(reference "R134")
+					(reference "R18")
 					(unit 1)
 				)
