File: ethernet.kicad_sch (KiCad schematic)
At the start: 27 parts, among them J6 RJ45_RB1-125B8G1A, U6 RTL8111H-CG-RH, U7 D3V3XA4B10LP, U8 D3V3XA4B10LP, Y1 25MHz

Commit message: Resolved some duplicate annotations
Parts:
- renumbered C12 to C47
Changed lines of the file:
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@@
 		(in_pos_files yes)
 		(dnp no)
-		(property "Reference" "C12"
+		(property "Reference" "C47"
 			(at 151.13 144.272 90)
 			(show_name no)
@@
 			(project "Carrier_Board"
 				(path "/e768274e-12f3-4f83-96f6-abb7638e0bc1/3ad1df68-0a03-497a-a7ee-c67c9856d4e6"
-					(reference "C12")
+					(reference "C47")
 					(unit 1)
 				)

Commit message: Found and fixed a routing mismatch in the gigabit RX TX pin mis assignment
Parts:
- U7, U8: now fitted
- renumbered C123 to C38, C125 to C39, C124 to C42, C126 to C43, C131 to C46, C46 to C48
Connections:
- net MDI2+: now also U7.4, U7.7 (NC); no longer U7.5, U7.6 (NC)
- net MDI2-: now also U7.5, U7.6 (NC); no longer U7.4, U7.7 (NC)
Changed lines of the file:
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@@
 		)
 	)
-	(label "MDI2+"
+	(label "MDI2-"
 		(at 256.54 54.61 0)
 		(effects
@@
 		)
 	)
-	(label "MDI2-"
+	(label "MDI2+"
 		(at 256.54 44.45 0)
 		(effects
@@
 	)
 	(hierarchical_label "GbE_PCIe_RX-"
-		(shape input)
+		(shape output)
 		(at 30.48 99.06 180)
 		(effects
@@
 		(in_pos_files yes)
 		(dnp no)
-		(property "Reference" "C131"
+		(property "Reference" "C46"
 			(at 151.384 106.68 90)
 			(show_name no)
@@
 			(project "Carrier_Board"
 				(path "/e768274e-12f3-4f83-96f6-abb7638e0bc1/3ad1df68-0a03-497a-a7ee-c67c9856d4e6"
-					(reference "C131")
+					(reference "C46")
 					(unit 1)
 				)
@@
 		(in_pos_files yes)
 		(dnp no)
-		(property "Reference" "C126"
+		(property "Reference" "C43"
 			(at 58.928 100.584 90)
 			(show_name no)
@@
 			(project "Carrier_Board"
 				(path "/e768274e-12f3-4f83-96f6-abb7638e0bc1/3ad1df68-0a03-497a-a7ee-c67c9856d4e6"
-					(reference "C126")
+					(reference "C43")
 					(unit 1)
 				)
@@
 		(on_board yes)
 		(in_pos_files yes)
-		(dnp yes)
+		(dnp no)
 		(fields_autoplaced yes)
 		(property "Reference" "U8"
@@
 		(in_pos_files yes)
 		(dnp no)
-		(property "Reference" "C125"
+		(property "Reference" "C39"
 			(at 58.928 98.044 90)
 			(show_name no)
@@
 			(project "Carrier_Board"
 				(path "/e768274e-12f3-4f83-96f6-abb7638e0bc1/3ad1df68-0a03-497a-a7ee-c67c9856d4e6"
-					(reference "C125")
+					(reference "C39")
 					(unit 1)
 				)
@@
 		(in_pos_files yes)
 		(dnp no)
-		(property "Reference" "C46"
+		(property "Reference" "C48"
 			(at 158.75 95.25 90)
 			(show_name no)
@@
 			(project "Carrier_Board"
 				(path "/e768274e-12f3-4f83-96f6-abb7638e0bc1/3ad1df68-0a03-497a-a7ee-c67c9856d4e6"
-					(reference "C46")
+					(reference "C48")
 					(unit 1)
 				)
@@
 		(in_pos_files yes)
 		(dnp no)
-		(property "Reference" "C123"
+		(property "Reference" "C38"
 			(at 58.928 92.964 90)
 			(show_name no)
@@
 			(project "Carrier_Board"
 				(path "/e768274e-12f3-4f83-96f6-abb7638e0bc1/3ad1df68-0a03-497a-a7ee-c67c9856d4e6"
-					(reference "C123")
+					(reference "C38")
 					(unit 1)
 				)
@@
 		(in_pos_files yes)
 		(dnp no)
-		(property "Reference" "C124"
+		(property "Reference" "C42"
 			(at 58.928 95.504 90)
 			(show_name no)
@@
 			(project "Carrier_Board"
 				(path "/e768274e-12f3-4f83-96f6-abb7638e0bc1/3ad1df68-0a03-497a-a7ee-c67c9856d4e6"
-					(reference "C124")
+					(reference "C42")
 					(unit 1)
 				)
@@
 		(on_board yes)
 		(in_pos_files yes)
-		(dnp yes)
+		(dnp no)
 		(fields_autoplaced yes)
 		(property "Reference" "U7"
