File: usb_2_3.kicad_sch (KiCad schematic)
At the start: 20 parts, among them J4 USB3_A_Stacked, J5 USB_A_Stacked, U3 D3V3XA4B10LP, U4 D3V3XA4B10LP, U5 D3V3XA4B10LP

Commit message: Fixed the net labels on U3 and routed them to the USB3 connector with correct impednece matching
Connections:
- net CON_USB3_SSTX_N: now also U3.4, U3.7 (NC)
- net CON_USB3_SSTX_P: now also U3.5, U3.6 (NC)
- net USB3_SSRX_N: no longer U3.4, U3.7 (NC)
- net USB3_SSRX_P: no longer U3.5, U3.6 (NC)
Changed lines of the file:
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@@
 		)
 	)
-	(label "CON_USB3_SSRX_P"
+	(label "CON_USB3_SSTX_P"
 		(at 80.01 133.35 0)
 		(effects
@@
 		)
 	)
-	(label "CON_USB3_SSRX_N"
+	(label "CON_USB3_SSTX_N"
 		(at 80.01 128.27 0)
 		(effects

Commit message: USB 3.0 routed and comleted
Connections:
- net CON_USB4_SSTX_N: no longer U5.1, U5.10 (NC), U5.4, U5.7 (NC)
- net CON_USB4_SSTX_P: no longer U5.2, U5.5, U5.6 (NC), U5.9 (NC)
- net USB3_SSRX_P: now also U5.4, U5.7 (NC)
- net USB4_SSRX_N: now also U5.2, U5.9 (NC)
- net USB4_SSRX_P: now also U5.1, U5.10 (NC)
- net USB_2_P1+: now also D5.1 (A1)
- net USB_2_P1-: now also D6.1 (A1)
- net USB_2_P2+: now also D7.1 (A1)
- net USB_2_P2-: now also D8.1 (A1)
- net USB_2_P3+: no longer D7.1 (A1)
- net USB_2_P3-: no longer D8.1 (A1)
- net USB_2_P5+: no longer D5.1 (A1)
- net USB_2_P5-: no longer D6.1 (A1)
- new net: U5.5, U5.6 (NC)
Changed lines of the file:
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@@
 	(generator_version "10.0")
 	(paper "A4")
-	(text_box "ESD protection for the USB 2.0 data lines"
+	(text_box "ESD protection for the USB 3.0 data lines"
 		(exclude_from_sim no)
 		(at 145.415 105.41 0)
@@
 		)
 	)
-	(label "CON_USB4_SSTX_N"
-		(at 54.61 166.37 180)
-		(effects
-			(font
-				(size 1.27 1.27)
-			)
-			(justify right bottom)
-		)
-	)
-	(label "CON_USB4_SSTX_P"
-		(at 54.61 171.45 180)
-		(effects
-			(font
-				(size 1.27 1.27)
-			)
-			(justify right bottom)
-		)
-	)
 	(label "CON_USB3_SSTX_P"
 		(at 80.01 133.35 0)
@@
 		)
 	)
-	(label "CON_USB2_D_P"
-		(at 170.18 129.54 180)
+	(label "CON_USB3_D_N"
+		(at 170.18 134.62 180)
+		(effects
+			(font
+				(size 1.27 1.27)
+			)
+			(justify right bottom)
+		)
+	)
+	(label "CON_USB4_SSRX_N"
+		(at 54.61 171.45 180)
 		(effects
 			(font
@@
 		)
 	)
+	(label "CON_USB4_D_N"
+		(at 170.18 124.46 180)
+		(effects
+			(font
+				(size 1.27 1.27)
+			)
+			(justify right bottom)
+		)
+	)
 	(label "CON_USB3_D_N"
 		(at 58.42 34.29 0)
@@
 		)
 	)
+	(label "CON_USB4_SSRX_P"
+		(at 54.61 166.37 180)
+		(effects
+			(font
+				(size 1.27 1.27)
+			)
+			(justify right bottom)
+		)
+	)
 	(label "CON_USB3_SSTX_N"
 		(at 80.01 128.27 0)
@@
 		)
 	)
-	(label "CON_USB4_SSTX_N"
-		(at 80.01 166.37 0)
-		(effects
-			(font
-				(size 1.27 1.27)
-			)
-			(justify left bottom)
-		)
-	)
 	(label "CON_USB3_SSRX_N"
 		(at 58.42 41.91 0)
@@
 		)
 	)
+	(label "CON_USB3_SSRX_P"
+		(at 80.01 166.37 0)
+		(effects
+			(font
+				(size 1.27 1.27)
+			)
+			(justify left bottom)
+		)
+	)
+	(label "CON_USB3_D_P"
+		(at 170.18 129.54 180)
+		(effects
+			(font
+				(size 1.27 1.27)
+			)
+			(justify right bottom)
+		)
+	)
+	(label "CON_USB3_SSRX_N"
+		(at 90.17 176.53 0)
+		(effects
+			(font
+				(size 1.27 1.27)
+			)
+			(justify left bottom)
+		)
+	)
 	(label "CON_USB4_SSTX_P"
 		(at 57.15 101.6 0)
@@
 		)
 	)
+	(label "CON_USB4_D_P"
+		(at 170.18 119.38 180)
+		(effects
+			(font
+				(size 1.27 1.27)
+			)
+			(justify right bottom)
+		)
+	)
 	(label "CON_USB1_D_N"
 		(at 185.42 50.8 0)
@@
 		)
 	)
-	(label "CON_USB1_D_P"
-		(at 170.18 119.38 180)
-		(effects
-			(font
-				(size 1.27 1.27)
-			)
-			(justify right bottom)
-		)
-	)
-	(label "CON_USB2_D_N"
-		(at 170.18 134.62 180)
-		(effects
-			(font
-				(size 1.27 1.27)
-			)
-			(justify right bottom)
-		)
-	)
-	(label "CON_USB1_D_N"
-		(at 170.18 124.46 180)
-		(effects
-			(font
-				(size 1.27 1.27)
-			)
-			(justify right bottom)
-		)
-	)
 	(label "CON_USB3_SSTX_N"
 		(at 58.42 49.53 0)
 		(effects
 			(font
-				(size 1.27 1.27)
-			)
-			(justify left bottom)
-		)
-	)
-	(label "CON_USB4_SSTX_P"
-		(at 80.01 171.45 0)
-		(effects
-			(font

Commit message: Routed USB 2 by myself
Connections:
- net USB_2_P3+: now also U4.2, U4.9 (NC); no longer U4.4, U4.7 (NC)
- net USB_2_P3-: now also U4.1, U4.10 (NC); no longer U4.5, U4.6 (NC)
- net USB_2_P5+: now also U4.5, U4.6 (NC); no longer U4.1, U4.10 (NC)
- net USB_2_P5-: now also U4.4, U4.7 (NC); no longer U4.2, U4.9 (NC)
Changed lines of the file:
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@@
-		)
-	)
-	(label "CON_USB2_D_N"
-		(at 207.01 76.2 0)
-		(effects
-			(font
-				(size 1.27 1.27)
-			)
-			(justify left bottom)
 		)
 	)
@@
 		)
 	)
+	(label "CON_USB2_D_P"
+		(at 181.61 76.2 180)
+		(effects
+			(font
+				(size 1.27 1.27)
+			)
+			(justify right bottom)
+		)
+	)
 	(label "CON_USB3_SSTX_N"
 		(at 80.01 128.27 0)
@@
 			)
 			(justify left bottom)
-		)
-	)
-	(label "CON_USB1_D_P"
-		(at 181.61 71.12 180)
-		(effects
-			(font
-				(size 1.27 1.27)
-			)
-			(justify right bottom)
 		)
 	)
@@
 		)
 	)
-	(label "CON_USB2_D_P"
+	(label "CON_USB1_D_N"
 		(at 207.01 71.12 0)
 		(effects
@@
 		)
 	)
-	(label "CON_USB1_D_N"
-		(at 181.61 76.2 180)
+	(label "CON_USB1_D_P"
+		(at 207.01 76.2 0)
 		(effects
 			(font
+				(size 1.27 1.27)
+			)
+			(justify left bottom)
+		)
+	)
+	(label "CON_USB2_D_N"
+		(at 181.61 71.12 180)
+		(effects
+			(font

Commit message: Updated umpopul;ated audio pins in sub audio sheet
Connections:
- net +5V: now also C30.2, F2.1, F3.1; no longer F2.2, F3.2, J5.1 (VBUS1), J5.5 (VBUS2)
- new net: F3.2, J5.5 (VBUS2)
- new net: F2.2, J5.1 (VBUS1)
Other:
- moved on the sheet: F2, F3
Changed lines of the file:
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@@
 	)
 	(junction
-		(at 199.39 40.64)
-		(diameter 0)
-		(color 0 0 0 0)
-	)
-	(junction
 		(at 80.01 78.74)
 		(diameter 0)
@@
 	)
 	(junction
-		(at 220.98 43.18)
-		(diameter 0)
-		(color 0 0 0 0)
-	)
-	(junction
-		(at 220.98 40.64)
+		(at 199.39 40.64)
 		(diameter 0)
 		(color 0 0 0 0)
@@
 	(wire
 		(pts
-			(xy 220.98 40.64) (xy 220.98 43.18)
-		)
-		(stroke
-			(width 0)
-			(type default)
-		)
-	)
-	(wire
-		(pts
 			(xy 45.72 101.6) (xy 87.63 101.6)
 		)
@@
 	(wire
 		(pts
-			(xy 220.98 40.64) (xy 227.33 40.64)
+			(xy 217.17 40.64) (xy 227.33 40.64)
 		)
 		(stroke
@@
 	(wire
 		(pts
-			(xy 210.82 40.64) (xy 220.98 40.64)
-		)
-		(stroke
-			(width 0)
-			(type default)
-		)
-	)
-	(wire
-		(pts
 			(xy 80.01 29.21) (xy 81.28 29.21)
 		)
@@
 	(wire
 		(pts
-			(xy 199.39 40.64) (xy 203.2 40.64)
+			(xy 199.39 29.21) (xy 199.39 40.64)
 		)
 		(stroke
@@
 	(wire
 		(pts
-			(xy 199.39 43.18) (xy 199.39 40.64)
+			(xy 199.39 40.64) (xy 209.55 40.64)
 		)
 		(stroke
@@
 	(wire
 		(pts
-			(xy 181.61 81.28) (xy 181.61 76.2)
+			(xy 199.39 43.18) (xy 199.39 40.64)
 		)
 		(stroke
@@
 	(wire
 		(pts
-			(xy 194.31 134.62) (xy 210.82 134.62)
+			(xy 181.61 81.28) (xy 181.61 76.2)
 		)
 		(stroke
@@
 	(wire
 		(pts
-			(xy 220.98 43.18) (xy 227.33 43.18)
+			(xy 194.31 134.62) (xy 210.82 134.62)
 		)
 		(stroke
@@
 	(wire
 		(pts
-			(xy 203.2 43.18) (xy 199.39 43.18)
+			(xy 209.55 43.18) (xy 199.39 43.18)
 		)
 		(stroke
@@
 	(wire
 		(pts
-			(xy 210.82 43.18) (xy 220.98 43.18)
+			(xy 217.17 43.18) (xy 227.33 43.18)
 		)
 		(stroke
@@
 	(wire
 		(pts
-			(xy 220.98 27.94) (xy 220.98 40.64)
-		)
-		(stroke
-			(width 0)
-			(type default)
-		)
-	)
-	(wire
-		(pts
 			(xy 170.18 48.26) (xy 227.33 48.26)
 		)
@@
 	(symbol
 		(lib_id "Device:Fuse")
-		(at 207.01 43.18 90)
+		(at 213.36 43.18 90)
 		(unit 1)
 		(body_style 1)
@@
 		(dnp no)
 		(property "Reference" "F3"
-			(at 201.93 44.45 90)
+			(at 208.28 44.45 90)
 			(show_name no)
 			(do_not_autoplace no)
@@
 		)
 		(property "Value" "6V/1A"
-			(at 213.868 44.704 90)
+			(at 220.218 44.704 90)
 			(show_name no)
 			(do_not_autoplace no)
@@
 		)
 		(property "Footprint" "A_HDJ_Library:Fuse_0805_2012Metric"
-			(at 207.01 44.958 90)
+			(at 213.36 44.958 90)
 			(hide yes)
 			(show_name no)
@@
 		)
 		(property "Datasheet" ""
-			(at 207.01 43.18 0)
+			(at 213.36 43.18 0)
 			(hide yes)
 			(show_name no)
@@
 		)
 		(property "Description" "Fuse"
-			(at 207.01 43.18 0)
+			(at 213.36 43.18 0)
 			(hide yes)
 			(show_name no)
@@
 		)
 		(property "Purpose" ""
-			(at 207.01 43.18 0)
+			(at 213.36 43.18 0)
 			(show_name no)
 			(do_not_autoplace no)
@@
 		)
 		(property "KLC_S3.3" ""
-			(at 207.01 43.18 90)
+			(at 213.36 43.18 90)
 			(hide yes)
 			(show_name no)
@@
 		)
 		(property "KLC_S4.1" ""
-			(at 207.01 43.18 90)
+			(at 213.36 43.18 90)
 			(hide yes)
 			(show_name no)
@@
 	(symbol
 		(lib_id "Device:Fuse")
-		(at 207.01 40.64 90)
+		(at 213.36 40.64 90)
 		(unit 1)
 		(body_style 1)
@@
 		(dnp no)
 		(property "Reference" "F2"
-			(at 201.93 39.624 90)
+			(at 208.28 39.624 90)
 			(show_name no)
 			(do_not_autoplace no)
@@
 		)
 		(property "Value" "6V/1A"
-			(at 213.614 39.116 90)
+			(at 219.964 39.116 90)
 			(show_name no)
 			(do_not_autoplace no)
@@
 		)
 		(property "Footprint" "A_HDJ_Library:Fuse_0805_2012Metric"
-			(at 207.01 42.418 90)
+			(at 213.36 42.418 90)
 			(hide yes)
 			(show_name no)
@@
 		)
 		(property "Datasheet" ""
-			(at 207.01 40.64 0)
+			(at 213.36 40.64 0)
 			(hide yes)
 			(show_name no)
@@
 		)
 		(property "Description" "Fuse"
-			(at 207.01 40.64 0)
+			(at 213.36 40.64 0)
 			(hide yes)
 			(show_name no)
@@
 		)
 		(property "Purpose" ""
-			(at 207.01 40.64 0)
+			(at 213.36 40.64 0)
 			(show_name no)
 			(do_not_autoplace no)
@@
 		)
 		(property "KLC_S3.3" ""
-			(at 207.01 40.64 90)
+			(at 213.36 40.64 90)
 			(hide yes)
 			(show_name no)
@@
 		)
 		(property "KLC_S4.1" ""
-			(at 207.01 40.64 90)
+			(at 213.36 40.64 90)
 			(hide yes)
 			(show_name no)
@@
 	(symbol
 		(lib_id "power:+5V")
-		(at 220.98 27.94 0)
+		(at 199.39 29.21 0)
 		(unit 1)
 		(body_style 1)
@@
 		(fields_autoplaced yes)
 		(property "Reference" "#PWR0169"
-			(at 220.98 31.75 0)
+			(at 199.39 33.02 0)
 			(hide yes)
 			(show_name no)
@@
 		)
 		(property "Value" "+5V"
-			(at 220.98 22.86 0)
+			(at 199.39 24.13 0)
 			(show_name no)
 			(do_not_autoplace no)
@@
 		)
 		(property "Footprint" ""
-			(at 220.98 27.94 0)
+			(at 199.39 29.21 0)
 			(hide yes)
 			(show_name no)
@@
 		)
 		(property "Datasheet" ""
-			(at 220.98 27.94 0)
+			(at 199.39 29.21 0)
 			(hide yes)
 			(show_name no)
@@
 		)
 		(property "Description" "Power symbol creates a global label with name \"+5V\""
-			(at 220.98 27.94 0)
+			(at 199.39 29.21 0)
 			(hide yes)
 			(show_name no)
